Commit message: Add new retargeting scripts for A1

File: resources/robots/a1/urdf/a1.urdf (robot description, URDF)
Before this commit: robot a1_description, 23 links, 22 joints
Joints:
- removed joint FL_calf_joint
- removed joint FL_foot_fixed
- removed joint FL_hip_fixed
- removed joint FL_hip_joint
- removed joint FL_thigh_joint
- removed joint FR_calf_joint
- removed joint FR_foot_fixed
- removed joint FR_hip_fixed
- removed joint FR_hip_joint
- removed joint FR_thigh_joint
- removed joint RL_calf_joint
- removed joint RL_foot_fixed
- removed joint RL_hip_fixed
- removed joint RL_hip_joint
- removed joint RL_thigh_joint
- removed joint RR_calf_joint
- removed joint RR_foot_fixed
- removed joint RR_hip_fixed
- removed joint RR_hip_joint
- removed joint RR_thigh_joint
- added joint leg0_FL_a_hip_joint: type revolute, parent trunk, child FL_hip, origin xyz=0.183 0.047 0 rpy=0 0 0, axis 1 0 0, limit lower=-1.2 upper=1.2 effort=20 velocity=52.4
- added joint leg0_FL_b_hip_fixed: type fixed, parent FL_hip, child FL_thigh_shoulder, origin xyz=0 0.081 0 rpy=0 0 0
- added joint leg0_FL_c_thigh_joint: type revolute, parent FL_hip, child FL_thigh, origin xyz=0 0.08505 0 rpy=0 0 0, axis 0 1 0, limit lower=-1.0471975512 upper=2.05 effort=55 velocity=28.6
- added joint leg0_FL_d_calf_joint: type revolute, parent FL_thigh, child FL_calf, origin xyz=0 0 -0.2 rpy=0 0 0, axis 0 1 0, limit lower=-2.69653369433 upper=-0.916297857297 effort=55 velocity=28.6
- added joint leg0_FL_e_foot_fixed: type fixed, parent FL_calf, child FL_foot, origin xyz=0 0 -0.2 rpy=0 0 0
- added joint leg1_FR_a_hip_joint: type revolute, parent trunk, child FR_hip, origin xyz=0.183 -0.047 0 rpy=0 0 0, axis 1 0 0, limit lower=-1.2 upper=1.2 effort=20 velocity=52.4
- added joint leg1_FR_b_hip_fixed: type fixed, parent FR_hip, child FR_thigh_shoulder, origin xyz=0 -0.081 0 rpy=0 0 0
- added joint leg1_FR_c_thigh_joint: type revolute, parent FR_hip, child FR_thigh, origin xyz=0 -0.08505 0 rpy=0 0 0, axis 0 1 0, limit lower=-1.0471975512 upper=2.05 effort=55 velocity=28.6
- added joint leg1_FR_d_calf_joint: type revolute, parent FR_thigh, child FR_calf, origin xyz=0 0 -0.2 rpy=0 0 0, axis 0 1 0, limit lower=-2.69653369433 upper=-0.916297857297 effort=55 velocity=28.6
- added joint leg1_FR_e_foot_fixed: type fixed, parent FR_calf, child FR_foot, origin xyz=0 0 -0.2 rpy=0 0 0
- added joint leg2_RL_a_hip_joint: type revolute, parent trunk, child RL_hip, origin xyz=-0.183 0.047 0 rpy=0 0 0, axis 1 0 0, limit lower=-1.2 upper=1.2 effort=20 velocity=52.4
- added joint leg2_RL_b_hip_fixed: type fixed, parent RL_hip, child RL_thigh_shoulder, origin xyz=0 0.081 0 rpy=0 0 0
- added joint leg2_RL_c_thigh_joint: type revolute, parent RL_hip, child RL_thigh, origin xyz=0 0.08505 0 rpy=0 0 0, axis 0 1 0, limit lower=-1.0471975512 upper=2.05 effort=55 velocity=28.6
- added joint leg2_RL_d_calf_joint: type revolute, parent RL_thigh, child RL_calf, origin xyz=0 0 -0.2 rpy=0 0 0, axis 0 1 0, limit lower=-2.69653369433 upper=-0.916297857297 effort=55 velocity=28.6
- added joint leg2_RL_e_foot_fixed: type fixed, parent RL_calf, child RL_foot, origin xyz=0 0 -0.2 rpy=0 0 0
- added joint leg3_RR_a_hip_joint: type revolute, parent trunk, child RR_hip, origin xyz=-0.183 -0.047 0 rpy=0 0 0, axis 1 0 0, limit lower=-1.2 upper=1.2 effort=20 velocity=52.4
- added joint leg3_RR_b_hip_fixed: type fixed, parent RR_hip, child RR_thigh_shoulder, origin xyz=0 -0.081 0 rpy=0 0 0
- added joint leg3_RR_c_thigh_joint: type revolute, parent RR_hip, child RR_thigh, origin xyz=0 -0.08505 0 rpy=0 0 0, axis 0 1 0, limit lower=-1.0471975512 upper=2.05 effort=55 velocity=28.6
- added joint leg3_RR_d_calf_joint: type revolute, parent RR_thigh, child RR_calf, origin xyz=0 0 -0.2 rpy=0 0 0, axis 0 1 0, limit lower=-2.69653369433 upper=-0.916297857297 effort=55 velocity=28.6
- added joint leg3_RR_e_foot_fixed: type fixed, parent RR_calf, child RR_foot, origin xyz=0 0 -0.2 rpy=0 0 0
